File: hardware/kicad/sbc-baseboard/target.kicad_sch (KiCad schematic)
At the start: 30 parts, among them J13 Console, J14 +5V_TGT out, J15 GPIO + I2C, U701 TXB0104PW, U702 TXB0108PW, U703 TXS0102DCU, U704 TPS26630RGE

Commit message: USB 2.0 differential pairs named for the router; USB net class; ports aligned
Every USB 2.0 data net is now <base>_P / <base>_N, the suffixes KiCad's PCB
editor pairs up: J1_D, J3_D, PORT1_D..PORT4_D on the receptacle side of each
ESD array; HUB_UP and HUB_DN1..HUB_DN7 at the hub; K64_USB and FTDI_USB at the
chips. All 15 pairs are complete with D+ on _P. The project file gains a USB
net class assigned by pattern (differential geometry to be set from the
stackup). The labels sit at wire ends with their text along the pair's own
wire; routes now run their last leg into a side pin as one wire so a label at
the pin end owns the stretch (Conn join=False keeps a shared stub where two
routes meet at one pin). The USB-A receptacles and their switches move down
1.27 mm so the pairs run straight from the ESD arrays, and the port ESD arrays
move left to make room for the labels. Netlist membership unchanged (356
nets); ERC, geometry, connectivity, layout and reproducibility gates all
clean.

Co-Authored-By: Claude Fable 5.1 <noreply@anthropic.com>
Changed lines of the file:
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@@
 		(pts
 			(xy 373.38 190.5)
-			(xy 372.11 190.5)
-		)
-		(stroke
-			(width 0)
-			(type default)
-		)
-	)
-	(wire
-		(pts
-			(xy 372.11 190.5)
 			(xy 374.65 190.5)
 		)
