File: hardware/kicad/sbc-baseboard/target.kicad_sch (KiCad schematic)
At the start: 30 parts, among them J13 Console, J14 +5V_TGT out, J15 GPIO + I2C, U701 TXB0104PW, U702 TXB0108PW, U703 TXS0102DCU, U704 TPS26630RGE

Commit message: The PD inlet and the two 5 V bucks go; a 2.5 mm barrel jack feeds one +5V rail through a reverse-polarity FET
Power in is a 5 V 4 A (20 W) adapter on a Kycon KLDX-0202-BC barrel
jack (J2, centre positive), clamped by an SMAJ5.0A, passed by a
DMP3013SFV P-channel MOSFET (body diode toward the rail, gate at GND,
9.5 mOhm) into +5V: two 47 uF and a 100 nF, an amber LED. The
STUSB4500, its I2C buffer and Qwiic programming header, the two
TPS54560B bucks and their islands, VBUS_IN, +5V_PORTS and +5V_TGT as
separate rails are gone; +5V feeds the port switches, the relays, the
FTDI switch, the 3V3 buck and the TPS26630 eFuse, whose output is the
switched target rail +5V_TGT, now limited to 3 A (RILIM 6.04k, the
datasheet's 18 kOhm.A / IOL). The K64's I2C0 and PD pins are freed.
Classes: PWR_4A (2.5 mm, 1.0 mm vias) for +5V and +5V_TGT in place of
PWR_6A; USB_VBUS_3A keeps the port and FTDI VBUS nets. The directives
anchor the FET behind the jack, drop the bucks' and the PD controller's
templates, and draw the one +5V rail on L4 from the jack to the eFuse.
ERC clean; the placement passes every gate, 481 connections to route.

Co-Authored-By: Claude Fable 5.1 <noreply@anthropic.com>
Parts:
- R708: value 3.65k 1% -> 6.04k 1%
Connections:
- net +5V_TGT_OUT is gone; now on net +5V_TGT: C710.1, J14.1 (Pin_1), R705.1, U704.17 (OUT), U704.18 (OUT)
- net +5V_TGT: no longer C708.1, C709.1, R703.1, U704.1 (IN), U704.2 (IN), U704.5 (IN_SYS)
- new net +5V: C708.1, C709.1, R703.1, U704.1 (IN), U704.2 (IN), U704.5 (IN_SYS)
Other:
- note added: "TPS26630: ILIM 6.04k -> 3 A (RILIM = 18 kOhm.A / IOL; 3.65k -> 5 A until 2026-10-10, when the 20 W inlet set the budget), UVLO 196k/75k -> 4.3 V, OVP/MODE/PGTH to GND (latch-off). IMON 20k -> 1.7 V at 3 A into PTB2."
- note removed: "TPS26630: ILIM 3.65k -> ~5 A, UVLO 196k/75k -> 4.3 V, OVP/MODE/PGTH to GND (latch-off). IMON 20k -> 2.8 V at 5 A into PTB2."
- moved on the sheet: R702, R703
Changed lines of the file:
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@@
 		)
 	)
-	(text "TPS26630: ILIM 3.65k -> ~5 A, UVLO 196k/75k -> 4.3 V, OVP/MODE/PGTH to GND (latch-off). IMON 20k -> 2.8 V at 5 A into PTB2."
+	(text "TPS26630: ILIM 6.04k -> 3 A (RILIM = 18 kOhm.A / IOL; 3.65k -> 5 A until 2026-10-10, when the 20 W inlet set the budget), UVLO 196k/75k -> 4.3 V, OVP/MODE/PGTH to GND (latch-off). IMON 20k -> 1.7 V at 3 A into PTB2."
 		(exclude_from_sim no)
 		(at 16 27.8 0)
@@
 			)
 		)
-		(property "Value" "+5V_TGT"
+		(property "Value" "+5V"
 			(at 238.76 170.18 0)
 			(show_name no)
@@
 		(pts
 			(xy 274.32 195.58)
-			(xy 233.68 195.58)
+			(xy 236.22 195.58)
 		)
 		(stroke
@@
 	(symbol
 		(lib_id "Device:R")
-		(at 233.68 203.2 0)
+		(at 236.22 203.2 0)
 		(unit 1)
 		(body_style 1)
@@
 		(fields_autoplaced no)
 		(property "Reference" "R702"
-			(at 231.14 201.93 0)
+			(at 233.68 201.93 0)
 			(show_name no)
 			(do_not_autoplace no)
@@
 		)
 		(property "Value" "75k"
-			(at 231.14 204.47 0)
+			(at 233.68 204.47 0)
 			(show_name no)
 			(do_not_autoplace no)
@@
 		)
 		(property "Footprint" "Resistor_SMD:R_0603_1608Metric"
-			(at 233.68 203.2 0)
+			(at 236.22 203.2 0)
 			(hide yes)
 			(show_name no)
@@
 		)
 		(property "Datasheet" "~"
-			(at 233.68 203.2 0)
+			(at 236.22 203.2 0)
 			(hide yes)
 			(show_name no)
@@
 		)
 		(property "Description" "Resistor"
-			(at 233.68 203.2 0)
+			(at 236.22 203.2 0)
 			(hide yes)
 			(show_name no)
@@
 	(wire
 		(pts
-			(xy 233.68 195.58)
-			(xy 233.68 199.39)
+			(xy 236.22 195.58)
+			(xy 236.22 199.39)
 		)
 		(stroke
@@
 	(wire
 		(pts
-			(xy 233.68 207.01)
-			(xy 233.68 209.55)
+			(xy 236.22 207.01)
+			(xy 236.22 209.55)
 		)
 		(stroke
@@
 	(symbol
 		(lib_id "power:GND")
-		(at 233.68 209.55 0)
+		(at 236.22 209.55 0)
 		(unit 1)
 		(body_style 1)
@@
 		(fields_autoplaced no)
 		(property "Reference" "#PWR08033"
-			(at 233.68 209.55 0)
+			(at 236.22 209.55 0)
 			(hide yes)
 			(show_name no)
@@
 		)
 		(property "Value" "GND"
-			(at 233.68 212.09 0)
+			(at 236.22 212.09 0)
 			(show_name no)
 			(do_not_autoplace no)
@@
 		)
 		(property "Footprint" ""
-			(at 233.68 209.55 0)
+			(at 236.22 209.55 0)
 			(hide yes)
 			(show_name no)
@@
 		)
 		(property "Datasheet" "~"
-			(at 233.68 209.55 0)
+			(at 236.22 209.55 0)
 			(hide yes)
 			(show_name no)
@@
 		)
 		(property "Description" "Power symbol creates a global label with name \"GND\" , ground"
-			(at 233.68 209.55 0)
+			(at 236.22 209.55 0)
 			(hide yes)
 			(show_name no)
@@
 	)
 	(junction
-		(at 233.68 195.58)
+		(at 236.22 195.58)
 		(diameter 0)
 		(color 0 0 0 0)
@@
 	(wire
 		(pts
-			(xy 233.68 195.58)
-			(xy 228.6 195.58)
+			(xy 236.22 195.58)
+			(xy 231.14 195.58)
 		)
 		(stroke
@@
 	(symbol
 		(lib_id "Device:R")
-		(at 228.6 187.96 0)
+		(at 231.14 187.96 0)
 		(unit 1)
 		(body_style 1)
@@
 		(fields_autoplaced no)
 		(property "Reference" "R703"
-			(at 226.06 186.69 0)
+			(at 228.6 186.69 0)
 			(show_name no)
 			(do_not_autoplace no)
@@
 		)
 		(property "Value" "196k"
-			(at 226.06 189.23 0)
+			(at 228.6 189.23 0)
 			(show_name no)
 			(do_not_autoplace no)
@@
 		)
 		(property "Footprint" "Resistor_SMD:R_0603_1608Metric"
-			(at 228.6 187.96 0)
+			(at 231.14 187.96 0)
 			(hide yes)
 			(show_name no)
@@
 		)
 		(property "Datasheet" "~"
-			(at 228.6 187.96 0)
+			(at 231.14 187.96 0)
 			(hide yes)
 			(show_name no)
@@
 		)
 		(property "Description" "Resistor"
-			(at 228.6 187.96 0)
+			(at 231.14 187.96 0)
 			(hide yes)
 			(show_name no)
@@
 	(wire
 		(pts
-			(xy 228.6 195.58)
-			(xy 228.6 191.77)
+			(xy 231.14 195.58)
+			(xy 231.14 191.77)
 		)
 		(stroke
@@
 	(wire
 		(pts
-			(xy 228.6 184.15)
-			(xy 228.6 181.61)
+			(xy 231.14 184.15)
+			(xy 231.14 181.61)
 		)
 		(stroke
@@
 	(symbol
 		(lib_id "power:+5V")
-		(at 228.6 181.61 0)
+		(at 231.14 181.61 0)
 		(unit 1)
 		(body_style 1)
@@
 		(fields_autoplaced no)
 		(property "Reference" "#PWR08034"
-			(at 228.6 181.61 0)
+			(at 231.14 181.61 0)
 			(hide yes)
 			(show_name no)
@@
 			)
 		)
-		(property "Value" "+5V_TGT"
-			(at 228.6 177.8 0)
+		(property "Value" "+5V"
+			(at 231.14 177.8 0)
 			(show_name no)
 			(do_not_autoplace no)
@@
 		)
 		(property "Footprint" ""
-			(at 228.6 181.61 0)
+			(at 231.14 181.61 0)
 			(hide yes)
 			(show_name no)
@@
 		)
 		(property "Datasheet" "~"
-			(at 228.6 181.61 0)
+			(at 231.14 181.61 0)
 			(hide yes)
 			(show_name no)
@@
 		)
 		(property "Description" "Power symbol creates a global label with name \"+5V\""
-			(at 228.6 181.61 0)
+			(at 231.14 181.61 0)
 			(hide yes)
 			(show_name no)
@@
 			)
 		)
-		(property "Value" "+5V_TGT"
+		(property "Value" "+5V"
 			(at 289.56 175.26 0)
 			(show_name no)
@@
 		)
 	)
-	(label "+5V_TGT_OUT"
+	(label "+5V_TGT"
 		(at 341.63 177.8 0)
 		(fields_autoplaced yes)
@@
 			)
 		)
-		(property "Value" "3.65k 1%"
+		(property "Value" "6.04k 1%"
 			(at 328.93 228.6 0)
 			(show_name no)
@@
 		)
 	)
-	(label "+5V_TGT_OUT"
+	(label "+5V_TGT"
 		(at 369.57 190.5 180)
 		(fields_autoplaced yes)
