File: hardware/kicad/sbc-baseboard/ethernet.kicad_sch (KiCad schematic)
At the start: 25 parts, among them J10 RJ45 magjack 10/100, U301 KSZ8081RNA, Y301 25MHz

Commit message: Clock sources flow downward; USB pairs ordered as on the ESD array
Every crystal is now drawn by one helper: the two XTAL lanes run out past
the side's route channels to two columns 7.62 mm apart, drop at right
angles through the crystal lying across them, on into one load capacitor
each and a shared GND rail with one GND symbol, which also takes the
crystal's ground pins. The capacitors no longer hang off the lanes beside
the hub with the crystal somewhere else; nothing crosses.

Library v0.2.2: USB pairs are listed D- above D+, the order of the lines
through a USBLC6 array, so J3/U202 now sit on the K64's USB rows with
straight wires and the hub's upstream routes no longer cross; the hub's XTAL
pins move to the bottom of its left column so the clock cluster hangs under
everything else there, with clear rows around VBUS_DET.

All sheets: ERC 0, contacts 0, merges 0, layout 0; connectivity unchanged.

Co-Authored-By: Claude Fable 5.1 <noreply@anthropic.com>
Parts:
- C304: value 22p -> 2u2
- C305: value 22p -> 100n
- C306: value 2u2 -> 22p
- C307: value 100n -> 22p
Connections:
- new net: C304.1, C305.1, U301.1 (VDD_1.2)
- new net: C306.1, U301.7 (XO), Y301.1
- new net: C307.1, U301.8 (XI), Y301.3

Commit message: Pairs laid as lanes, the rails as L3 regions, the Ethernet pairs named: the board ready for the bulk router
All sixteen USB 2.0 pair segments and the two Ethernet MDI pairs are laid
by the standard's placer from pair lanes in gen/layout.py: members at the
class geometry, escapes at the pads, the USB-C receptacles' doubled pads
bridged behind their rows, two pairs passing under the port pairs on the
bottom, every pair matched to within 0.25 mm, no crossings (the port
arrays and the J3 array use the house symbol drawn with I/O2 on top, the
K64's USB pins wired to its rows). J4 and J5 trade places so each stack's
pairs reach the hub row they are wired to. The ESD arrays, the series
parts and the SWD header are anchored for the lanes. The rails are
regions on In2.Cu at distinct priorities over a 3V3 base. The Ethernet
MDI pairs are named ETH_TD/RD and classed ETH (100 ohm). DRC: the 12
documented errors, no warnings but the unfilled rail islands; 499
connections for the bulk router (gen/pcb.py --route), which is running.

Co-Authored-By: Claude Fable 5.1 <noreply@anthropic.com>
Connections:
- net ETH_RD_N: now reaches J10.6 (RD-), U301.3 (RXM)
- net ETH_RD_P: now reaches J10.3 (RD+), U301.4 (RXP)
- net ETH_TD_N: now reaches J10.2 (TD-), U301.5 (TXM)
- net ETH_TD_P: now reaches J10.1 (TD+), U301.6 (TXP)
Changed lines of the file:
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@@
+		)
+	)
+	(label "ETH_TD_P"
+		(at 182.88 114.3 0)
+		(fields_autoplaced yes)
+		(effects
+			(font
+				(size 1.27 1.27)
+			)
+			(justify left bottom)
+		)
+	)
+	(label "ETH_TD_N"
+		(at 182.88 111.76 0)
+		(fields_autoplaced yes)
+		(effects
+			(font
+				(size 1.27 1.27)
+			)
+			(justify left bottom)
+		)
+	)
+	(label "ETH_RD_P"
+		(at 182.88 106.68 0)
+		(fields_autoplaced yes)
+		(effects
+			(font
+				(size 1.27 1.27)
+			)
+			(justify left bottom)
+		)
+	)
+	(label "ETH_RD_N"
+		(at 182.88 104.14 0)
+		(fields_autoplaced yes)
+		(effects
+			(font
+				(size 1.27 1.27)
+			)
+			(justify left bottom)
 		)
 	)
