File: hardware/kicad/sbc-baseboard/daplink.kicad_sch (KiCad schematic)
At the start: 15 parts, among them J601 SWD (K20), SW601 DAP RESET, U601 MK20DX128VFM5, Y601 8MHz

Commit message: Clock sources flow downward; USB pairs ordered as on the ESD array
Every crystal is now drawn by one helper: the two XTAL lanes run out past
the side's route channels to two columns 7.62 mm apart, drop at right
angles through the crystal lying across them, on into one load capacitor
each and a shared GND rail with one GND symbol, which also takes the
crystal's ground pins. The capacitors no longer hang off the lanes beside
the hub with the crystal somewhere else; nothing crosses.

Library v0.2.2: USB pairs are listed D- above D+, the order of the lines
through a USBLC6 array, so J3/U202 now sit on the K64's USB rows with
straight wires and the hub's upstream routes no longer cross; the hub's XTAL
pins move to the bottom of its left column so the clock cluster hangs under
everything else there, with clear rows around VBUS_DET.

All sheets: ERC 0, contacts 0, merges 0, layout 0; connectivity unchanged.

Co-Authored-By: Claude Fable 5.1 <noreply@anthropic.com>
Parts:
- C601: value 18p -> 100n
- C602: value 18p -> 2u2
- C604: value 2u2 -> 100n
- C605: value 100n -> 2u2
- C606: value 100n -> 18p
- C607: value 2u2 -> 18p
Connections:
- net +5V_PORTS: now also C605.1; no longer C607.1
- net K20_3V3: now also C602.1, C603.1; no longer C605.1, C606.1
- net at J601.10 (~{RESET}), R602.2, SW601.1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: now also C601.1; no longer C603.1
- new net: C606.1, U601.17 (PTA18), Y601.1
- new net: C607.1, U601.18 (PTA19), Y601.3
- new net: J601.4 (SWCLK/TCK), U601.12 (PTA0)

Commit message: Reset circuits flow downward: pull-up, capacitor and button in one cluster
A Reset attachment in the fan engine draws the network at the lane end, top to
bottom: rail symbol, pull-up, the node row where the lane arrives, the capacitor
straight below in the same column, one GND under it; a push button hangs from
the lane one column nearer the hub and shares the GND rail. It declares its
reaches, so the spread and slide passes keep the neighbouring rows clear. Used
for the K64 (RESET), the USB2517 and the K20 (DAP RESET); the K20's SWD header
takes the K20_RESET_N label instead of a fourth wire into the node. Netlist
membership unchanged (356 nets); ERC, geometry, connectivity and layout gates
all at zero.

Co-Authored-By: Claude Fable 5.1 <noreply@anthropic.com>
Connections:
- net GND: now also SW601.1; no longer SW601.2
- net K20_RESET_N: now reaches C601.1, J601.10 (~{RESET}), R602.2, U601.19 (~{RESET})
- net K20_RESET_N: now also SW601.2; no longer SW601.1

Commit message: USB 2.0 differential pairs named for the router; USB net class; ports aligned
Every USB 2.0 data net is now <base>_P / <base>_N, the suffixes KiCad's PCB
editor pairs up: J1_D, J3_D, PORT1_D..PORT4_D on the receptacle side of each
ESD array; HUB_UP and HUB_DN1..HUB_DN7 at the hub; K64_USB and FTDI_USB at the
chips. All 15 pairs are complete with D+ on _P. The project file gains a USB
net class assigned by pattern (differential geometry to be set from the
stackup). The labels sit at wire ends with their text along the pair's own
wire; routes now run their last leg into a side pin as one wire so a label at
the pin end owns the stretch (Conn join=False keeps a shared stub where two
routes meet at one pin). The USB-A receptacles and their switches move down
1.27 mm so the pairs run straight from the ESD arrays, and the port ESD arrays
move left to make room for the labels. Netlist membership unchanged (356
nets); ERC, geometry, connectivity, layout and reproducibility gates all
clean.

Co-Authored-By: Claude Fable 5.1 <noreply@anthropic.com>
Connections:
- net HUB_DN1_DM renamed HUB_DN1_N
- net HUB_DN1_DP renamed HUB_DN1_P
Other:
- moved on the sheet: C601, C606, C607, R602, SW601, Y601

Commit message: Nothing drawn over anything else; FTDI Friend header; DAPLink per FRDM-K64F; 90 ohm USB class
Geometry gate now also reports two wires sharing a stretch, and is at zero on
every sheet. Routes into a stacked connector from one side take staggered
columns and rows; the signal relays are flipped so COM meets the header's
first pin without crossings; the opto-isolator moves above the passthrough
wires and taps the relay's COM lane; a tag before a route ends at the route's
target; routes into joined pins end at the join; the K64's VREGIN diode taps
the VBUS lane beside the ESD's stub; symbol mirrors are applied after
rotation, as KiCad does.

FT231X: the 3V3OUT lane stays on its pin row with its capacitor far out, clear
of the VCC decoupling; J9 mirrors the Adafruit FTDI Friend (VCC 5 V and pin 6
RTS by default on bridged solder jumpers; the first pass had left J9's VCC on
an open jumper only).

DAPLink K20, verified against DAPLink k20dx and the FRDM-K64F OpenSDA circuit:
PTC7 (SWDIO_IN) joins the SWDIO net, 33 R series resistors on the K20's USB
pair (K20_USB_P/N), notes and spec questions 12 and 14 resolved.

USB net class: 0.35 mm / 0.20 mm for 90 ohm on Advanced Circuits' standard
4-layer 62 mil stackup (spec section 8a). ERC 0, geometry 0, merges 0, layout
0, builds reproducible.

Co-Authored-By: Claude Fable 5.1 <noreply@anthropic.com>
Parts:
- added R604: 10k, Resistor_SMD:R_0603_1608Metric, symbol Device:R
- added R605: 470, Resistor_SMD:R_0603_1608Metric, symbol Device:R
- R602: value 10k -> 33
- R603: value 470 -> 33
Connections:
- net HUB_DN1_N: now also R603.2; no longer U601.4 (USB0_DM)
- net HUB_DN1_P: now also R602.2; no longer U601.3 (USB0_DP)
- net K20_3V3: now also R604.1, R605.2; no longer R602.1, R603.2
- net K20_RESET_N: now also R604.2; no longer R602.2
- net SWDIO: now also U601.28 (PTC7)
- net at D601.2 (A): now also R605.1; no longer R603.1
- new net K20_USB_N: R603.1, U601.4 (USB0_DM)
- new net K20_USB_P: R602.1, U601.3 (USB0_DP)
- no-connect marks 14 -> 13
Other:
- note added: "PTC7 (SWDIO_IN) ties to SWDIO, 33 R in series with USB D+/D- (FRDM R20/R22). No level shifters: the K64 target is 3.3 V like the K20."
- note added: "UART1 PTC3/PTC4 bridges to the K64 UART0 (CDC console). Pins verified against DAPLink k20dx IO_Config.h and the FRDM-K64F OpenSDA circuit:"
- note removed: "UART1 PTC3/PTC4 bridges to the K64 UART0 (CDC console). Verify against DAPLink source/hic_hal/freescale/k20dx/IO_Config.h."
- moved on the sheet: C601, C602, C606, C607, R601, R602, R603, SW601, Y601

Commit message: The PD inlet and the two 5 V bucks go; a 2.5 mm barrel jack feeds one +5V rail through a reverse-polarity FET
Power in is a 5 V 4 A (20 W) adapter on a Kycon KLDX-0202-BC barrel
jack (J2, centre positive), clamped by an SMAJ5.0A, passed by a
DMP3013SFV P-channel MOSFET (body diode toward the rail, gate at GND,
9.5 mOhm) into +5V: two 47 uF and a 100 nF, an amber LED. The
STUSB4500, its I2C buffer and Qwiic programming header, the two
TPS54560B bucks and their islands, VBUS_IN, +5V_PORTS and +5V_TGT as
separate rails are gone; +5V feeds the port switches, the relays, the
FTDI switch, the 3V3 buck and the TPS26630 eFuse, whose output is the
switched target rail +5V_TGT, now limited to 3 A (RILIM 6.04k, the
datasheet's 18 kOhm.A / IOL). The K64's I2C0 and PD pins are freed.
Classes: PWR_4A (2.5 mm, 1.0 mm vias) for +5V and +5V_TGT in place of
PWR_6A; USB_VBUS_3A keeps the port and FTDI VBUS nets. The directives
anchor the FET behind the jack, drop the bucks' and the PD controller's
templates, and draw the one +5V rail on L4 from the jack to the eFuse.
ERC clean; the placement passes every gate, 481 connections to route.

Co-Authored-By: Claude Fable 5.1 <noreply@anthropic.com>
Connections:
- net +5V_PORTS renamed +5V
Other:
- note added: "MK20DX128VFM5 running DAPLink (k20dx HIC), powered from +5V through its own USB regulator (VOUT33 -> VDD)."
- note removed: "MK20DX128VFM5 running DAPLink (k20dx HIC), powered from +5V_PORTS through its own USB regulator (VOUT33 -> VDD)."
Changed lines of the file:
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@@
 		)
 	)
-	(text "MK20DX128VFM5 running DAPLink (k20dx HIC), powered from +5V_PORTS through its own USB regulator (VOUT33 -> VDD)."
+	(text "MK20DX128VFM5 running DAPLink (k20dx HIC), powered from +5V through its own USB regulator (VOUT33 -> VDD)."
 		(exclude_from_sim no)
 		(at 16 19.7 0)
@@
 			)
 		)
-		(property "Value" "+5V_PORTS"
+		(property "Value" "+5V"
 			(at 152.4 55.88 0)
 			(show_name no)
