File: hardware/kicad/sbc-baseboard/hub.kicad_sch (KiCad schematic)
At the start: 84 parts, among them J1 USB-C upstream, J4 USB-A x2, J5 USB-A x2, U401 USBLC6-2SC6, U402 USB2517, U403 TPS2553DBV, U404 TPS2553DBV, U405 TPS2553DBV, U406 TPS2553DBV, U407 TPS2553DBV, U408 USBLC6-2SC6, U409 USBLC6-2SC6, U410 USBLC6-2SC6, U411 USBLC6-2SC6, Y401 24MHz

Commit message: The PD inlet and the two 5 V bucks go; a 2.5 mm barrel jack feeds one +5V rail through a reverse-polarity FET
Power in is a 5 V 4 A (20 W) adapter on a Kycon KLDX-0202-BC barrel
jack (J2, centre positive), clamped by an SMAJ5.0A, passed by a
DMP3013SFV P-channel MOSFET (body diode toward the rail, gate at GND,
9.5 mOhm) into +5V: two 47 uF and a 100 nF, an amber LED. The
STUSB4500, its I2C buffer and Qwiic programming header, the two
TPS54560B bucks and their islands, VBUS_IN, +5V_PORTS and +5V_TGT as
separate rails are gone; +5V feeds the port switches, the relays, the
FTDI switch, the 3V3 buck and the TPS26630 eFuse, whose output is the
switched target rail +5V_TGT, now limited to 3 A (RILIM 6.04k, the
datasheet's 18 kOhm.A / IOL). The K64's I2C0 and PD pins are freed.
Classes: PWR_4A (2.5 mm, 1.0 mm vias) for +5V and +5V_TGT in place of
PWR_6A; USB_VBUS_3A keeps the port and FTDI VBUS nets. The directives
anchor the FET behind the jack, drop the bucks' and the PD controller's
templates, and draw the one +5V rail on L4 from the jack to the eFuse.
ERC clean; the placement passes every gate, 481 connections to route.

Co-Authored-By: Claude Fable 5.1 <noreply@anthropic.com>
Connections:
- net +5V_PORTS renamed +5V
Other:
- note added: "Current: PORTn_VBUS and FTDI_VBUS are laid out for 3 A each (class USB_VBUS_3A, 2 mm traces); +5V feeds them from the 4 A inlet (class PWR_4A, 2.5 mm traces or pours)"
- note removed: "Current: PORTn_VBUS and FTDI_VBUS are laid out for 3 A each (class USB_VBUS_3A, 2 mm traces); +5V_PORTS feeds them at up to 6 A (PWR_6A)."
Changed lines of the file:
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@@
 		)
 	)
-	(text "Current: PORTn_VBUS and FTDI_VBUS are laid out for 3 A each (class USB_VBUS_3A, 2 mm traces); +5V_PORTS feeds them at up to 6 A (PWR_6A)."
+	(text "Current: PORTn_VBUS and FTDI_VBUS are laid out for 3 A each (class USB_VBUS_3A, 2 mm traces); +5V feeds them from the 4 A inlet (class PWR_4A, 2.5 mm traces or pours)"
 		(exclude_from_sim no)
 		(at 16 35.9 0)
@@
 			)
 		)
-		(property "Value" "+5V_PORTS"
+		(property "Value" "+5V"
 			(at 290.83 52.07 0)
 			(show_name no)
@@
 			)
 		)
-		(property "Value" "+5V_PORTS"
+		(property "Value" "+5V"
 			(at 290.83 102.87 0)
 			(show_name no)
@@
 			)
 		)
-		(property "Value" "+5V_PORTS"
+		(property "Value" "+5V"
 			(at 290.83 153.67 0)
 			(show_name no)
@@
 			)
 		)
-		(property "Value" "+5V_PORTS"
+		(property "Value" "+5V"
 			(at 290.83 204.47 0)
 			(show_name no)
@@
 			)
 		)
-		(property "Value" "+5V_PORTS"
+		(property "Value" "+5V"
 			(at 177.8 240.03 0)
 			(show_name no)
