File: hardware/kicad/sbc-baseboard/power.kicad_sch (KiCad schematic)
At the start: 86 parts, among them J17 Qwiic PD, J2 USB-C PD in, Q101 2N7002, Q102 2N7002, U101 STUSB4500QTR, U102 PCA9517A, U103 TPS54560BDDA, U104 TPS54560BDDA, U105 TPS62823DLC

Commit message: The PD inlet and the two 5 V bucks go; a 2.5 mm barrel jack feeds one +5V rail through a reverse-polarity FET
Power in is a 5 V 4 A (20 W) adapter on a Kycon KLDX-0202-BC barrel
jack (J2, centre positive), clamped by an SMAJ5.0A, passed by a
DMP3013SFV P-channel MOSFET (body diode toward the rail, gate at GND,
9.5 mOhm) into +5V: two 47 uF and a 100 nF, an amber LED. The
STUSB4500, its I2C buffer and Qwiic programming header, the two
TPS54560B bucks and their islands, VBUS_IN, +5V_PORTS and +5V_TGT as
separate rails are gone; +5V feeds the port switches, the relays, the
FTDI switch, the 3V3 buck and the TPS26630 eFuse, whose output is the
switched target rail +5V_TGT, now limited to 3 A (RILIM 6.04k, the
datasheet's 18 kOhm.A / IOL). The K64's I2C0 and PD pins are freed.
Classes: PWR_4A (2.5 mm, 1.0 mm vias) for +5V and +5V_TGT in place of
PWR_6A; USB_VBUS_3A keeps the port and FTDI VBUS nets. The directives
anchor the FET behind the jack, drop the bucks' and the PD controller's
templates, and draw the one +5V rail on L4 from the jack to the eFuse.
ERC clean; the placement passes every gate, 481 connections to route.

Co-Authored-By: Claude Fable 5.1 <noreply@anthropic.com>
Parts:
- removed C108, C109, C110: 100n, Capacitor_SMD:C_0603_1608Metric, symbol Device:C
- removed C111, C116, C120, C125: 100n/50V, Capacitor_SMD:C_0603_1608Metric, symbol Device:C
- removed C112, C113, C121, C122: 10u/50V, Capacitor_SMD:C_1210_3225Metric, symbol Device:C
- removed C114, C123: 47p, Capacitor_SMD:C_0603_1608Metric, symbol Device:C
- removed C115, C124: 4n7, Capacitor_SMD:C_0603_1608Metric, symbol Device:C
- removed C117, C118, C126, C127: 47u/10V, Capacitor_SMD:C_1210_3225Metric, symbol Device:C
- removed C119, C128: 100u/10V, Capacitor_SMD:CP_Elec_8x10.5, symbol Device:C_Polarized
- removed C129: 10u, Capacitor_SMD:C_0805_2012Metric, symbol Device:C
- removed C130, C131: 22u, Capacitor_SMD:C_0805_2012Metric, symbol Device:C
- removed C132: 120p, Capacitor_SMD:C_0603_1608Metric, symbol Device:C
- removed D104: ESDA25W, Diode_SMD:D_SOD-523, symbol Device:D_TVS
- removed D105, D109, D111, D113, D114: LED AMBER, LED_SMD:LED_0603_1608Metric, symbol Device:LED
- removed D106, D107: PESD5V0S1UL, Diode_SMD:D_SOD-882, symbol Diode:PESD5V0S1UL
- removed D108: BZT52C5V1, Diode_SMD:D_SOD-123, symbol Device:D_Zener
- removed D110, D112: B560C, Diode_SMD:D_SMA, symbol Device:D_Schottky
- removed J17: Qwiic PD, Connector_JST:JST_SH_BM04B-SRSS-TB_1x04-1MP_P1.00mm_Vertical, symbol Connector_Generic:Conn_01x04
- removed L102: 10u/6A, Inductor_SMD:L_Coilcraft_XAL7020-102, symbol Device:L
- removed L103: 470n/4A, Inductor_SMD:L_1210_3225Metric, symbol Device:L
- removed Q102: 2N7002, Package_TO_SOT_SMD:SOT-23, symbol Transistor_FET:2N7002
- removed R106, R109, R110: 10k, Resistor_SMD:R_0603_1608Metric, symbol Device:R
- removed R107, R111, R112, R113, R115, R127: 100k, Resistor_SMD:R_0603_1608Metric, symbol Device:R
- removed R108: 470, Resistor_SMD:R_1206_3216Metric, symbol Device:R
- removed R114, R126: 470, Resistor_SMD:R_0603_1608Metric, symbol Device:R
- removed R116, R121: 243k, Resistor_SMD:R_0603_1608Metric, symbol Device:R
- removed R117, R122: 16.9k, Resistor_SMD:R_0603_1608Metric, symbol Device:R
- removed R118, R123: 9.76k, Resistor_SMD:R_0603_1608Metric, symbol Device:R
- removed R119, R124: 51.1k, Resistor_SMD:R_0603_1608Metric, symbol Device:R
- removed R120, R125: 1k, Resistor_SMD:R_0603_1608Metric, symbol Device:R
- removed R128: 453k, Resistor_SMD:R_0603_1608Metric, symbol Device:R
- removed U101: STUSB4500QTR, Package_DFN_QFN:QFN-24-1EP_4x4mm_P0.5mm_EP2.7x2.7mm, symbol Interface_USB:STUSB4500QTR
- removed U102: PCA9517A, Package_SO:TSSOP-8_4.4x3mm_P0.65mm, symbol calico-ic:PCA9517A
- removed U103, U104: TPS54560BDDA, Package_SO:HSOP-8-1EP_3.9x4.9mm_P1.27mm_EP2.41x3.1mm, symbol calico-ic:TPS54560BDDA
- C101, C102: value 10u/50V -> 47u/10V
- C103: value 100n/50V -> 100n
- C104: value 1u/50V -> 10u
- C105, C106: value 1u -> 22u; footprint Capacitor_SMD:C_0603_1608Metric -> Capacitor_SMD:C_0805_2012Metric
- C107: value 1u -> 120p
- D101: value BAT54C -> SMAJ5.0A; footprint Package_TO_SOT_SMD:SOT-23 -> Diode_SMD:D_SMA; symbol Diode:BAT54C -> Device:D_Zener
- D102: value SMAJ24A -> LED AMBER; footprint Diode_SMD:D_SMA -> LED_SMD:LED_0603_1608Metric; symbol Device:D_Zener -> Device:LED
- D103: value ESDA25W -> LED AMBER; footprint Diode_SMD:D_SOD-523 -> LED_SMD:LED_0603_1608Metric; symbol Device:D_TVS -> Device:LED
- J2: value USB-C PD in -> 5 V in, 2.5 mm; footprint calico:USB_C_Receptacle_GCT_USB4105-xx-A_16P_TopMnt_Horizontal_PegClear -> Connector_BarrelJack:BarrelJack_Kycon_KLDX-0202-xC_Horizontal; symbol Connector:USB_C_Receptacle_USB2.0_16P -> Connector:Barrel_Jack_Switch
- L101: value 10u/6A -> 470n/4A; footprint Inductor_SMD:L_Coilcraft_XAL7020-102 -> Inductor_SMD:L_1210_3225Metric
- Q101: value 2N7002 -> DMP3013SFV; footprint Package_TO_SOT_SMD:SOT-23 -> Package_SON:Diodes_PowerDI3333-8; symbol Transistor_FET:2N7002 -> Transistor_FET:DMP3013SFV
- R101: value 10k -> 1k
- R102: value 10k -> 100k
- R103: value 1k -> 470
- R104: value 4.7k -> 100k
- R105: value 4.7k -> 453k
Connections:
- net BUCK_EN is gone; now on net +5V: Q101.3 (S)
- net PD_EN_GATE is gone; now on net +5V: Q101.1 (S)
- net PD_SCL is gone; now on net GND: R104.2
- net PD_SDA is gone; now on an unnamed net: R105.2
- net +3V3: now also C105.1, C106.1, C107.1, L101.2, R103.1, R105.1; no longer D101.1
- net GND: now also D101.2 (A), D102.1 (K), J2.2; no longer C107.2, D102.2 (A), J2.A1 (GND), J2.A12 (GND), J2.B1 (GND), J2.B12 (GND), J2.SH (SHIELD), Q101.2 (S)
- net at U105.2 (FB): now also C107.2, R104.1
- net at L101.1: now also U105.6 (SW)
- net at D103.2 (A): now also R103.2; no longer J2.A5 (CC1)
- net at R101.2: now also D102.2 (A)
- net at R102.1: now also Q101.4 (G)
- removed net +3V3_PD: D101.3, R104.1, R105.1
- removed net +3V3_PRG: C107.1, D101.2
- net +5V_PORTS renamed +5V
- net +5V: now also C101.1, C102.1, C103.1, C104.1, Q101.2 (S), R101.1; no longer L101.2
- removed net VBUS_IN: C101.1, C102.1, C103.1, C104.1, D102.1 (K), J2.A4 (VBUS), J2.A9 (VBUS), J2.B4 (VBUS), J2.B9 (VBUS), R101.1, R103.2
- new net: D101.1 (K), J2.1, Q101.5 (D)
- no-connect marks 13 -> 3
Other:
- note added: "+5V is laid out for 4 A (class PWR_4A, 2.5 mm or pours); +5V_TGT leaves the eFuse at up to 3 A in the same class."
- note added: "5 V bucks until then). SMAJ5.0A clamps the inlet; Q101, a P-channel MOSFET with its body diode toward the rail and its"
- note added: "J2: 2.5 x 5.5 mm barrel jack, centre positive, for a 5 V 4 A (20 W) adapter (2026-10-10; a USB-C PD inlet with two"
- note added: "board (0.5 A) can ask for more together; firmware keeps the budget (docs/hardware-spec.md section 4)."
- note added: "gate at GND, blocks reverse polarity at 9.5 mOhm. No series fuse: the adapter limits the inlet, the eFuse the target rail,"
- note added: "the TPS2553s the ports. The adapter's 4 A is the only limit on the sum: the ports (4 x 1.1 A), the target rail (3 A) and the"
- note removed: "-> EN low -> bucks off. Contract valid -> VBUS_EN_SNK low"
- note removed: "-> Q101 off -> EN floats high (internal pull-up) -> bucks on."
- note removed: "A programmer on J17 pulls PCA_EN low through Q102: the K64 is disconnected from the PD bus in hardware."
- note removed: "BUCK_EN: VBUS_EN_SNK released (no contract) -> Q101 on"
- note removed: "Current: VBUS_IN is laid out for 3 A (class USB_VBUS_3A, 2 mm); +5V_PORTS and +5V_TGT for 6 A (class PWR_6A, 4 mm or pours)."
- note removed: "FB 51.1k/9.76k -> 5.0 V. COMP 16.9k / 4.7n / 47p and the B560C are the"
- note removed: "J17 (Qwiic) programs the STUSB4500 NVM and powers it through VSYS when the board is dead."
- note removed: "J2 is a PD sink only (no data). STUSB4500 negotiates from NVM; VBUS_EN_SNK gates the 5 V bucks through Q101,"
- note removed: "PCA9517A: A side = PD segment (+3V3_PD, diode-OR of +3V3 and the programmer), B side = K64 I2C0."
- note removed: "TPS54560B: non-synchronous, 4.5-60 V in, 5 A. fsw 400 kHz (RT 243k)."
- note removed: "The zener keeps the gate under 5.1 V at 20 V VBUS."
- note removed: "datasheet's 5 V / 400 kHz design example (141 uF ceramic out, as here)."
- note removed: "so the rails only come up once a sink contract (or plain Type-C 5 V) is valid. No series VBUS FET."
- title: Power: PD inlet, programming header, bus buffer, three bucks -> Power: 5 V barrel inlet, input protection, 3V3 buck
- moved on the sheet: C101, C102, C103, C104, C105, C106, C107, L101, Q101, R101, R102, R103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

Commit message: The documents, the block diagram and the placed board for the barrel-jack inlet; 100 uF of bulk at the inlet
The specification (block diagram, connectors, parts, power tree and
budget at 20 W, pin budget, open questions, current pathways), the
README and the block diagram, the layout directives, guidelines and
reference-design review, the KiCad README and the protocol describe the
barrel inlet, the one +5V rail and the 3 A target rail; the PD inlet,
its controller, header and buffer and the two bucks remain as dated
history. A 100 uF electrolytic joins the two 47 uF at the inlet: the
hub's downstream ports want 120 uF on their rail, which buck 1's 194 uF
had given. Three older contradictions in the specification are settled
from the generator and the BOM: one FET per relay coil (2N7002 for the
signal relays, AO3400A for the power relay), the DAPLink on hub port 1,
the USB-A ports on hub ports 4 to 7. The board is committed placed and
unrouted (the route was stopped at the owner's request before it
finished): 271 parts, 480 connections, DRC clean.

Co-Authored-By: Claude Fable 5.1 <noreply@anthropic.com>
Parts:
- added C108: 120p, Capacitor_SMD:C_0603_1608Metric, symbol Device:C
- C103: value 100n -> 100u/10V; footprint Capacitor_SMD:C_0603_1608Metric -> Capacitor_SMD:CP_Elec_8x10.5; symbol Device:C -> Device:C_Polarized
- C104: value 10u -> 100n; footprint Capacitor_SMD:C_0805_2012Metric -> Capacitor_SMD:C_0603_1608Metric
- C105: value 22u -> 10u
- C107: value 120p -> 22u; footprint Capacitor_SMD:C_0603_1608Metric -> Capacitor_SMD:C_0805_2012Metric
Connections:
- net +3V3: now also C108.1; no longer C105.1
- net +5V: now also C105.1
- net GND: now also C107.2
- net at R104.1, R105.2, U105.2 (FB): now also C108.2; no longer C107.2
Other:
- note added: "No series fuse: the adapter limits the inlet, the eFuse the target rail,"
- note added: "gate at GND, blocks reverse polarity at 9.5 mOhm. 2 x 47 uF + 100 uF bulk behind it: the hub's downstream ports want 120 uF."
- note removed: "gate at GND, blocks reverse polarity at 9.5 mOhm. No series fuse: the adapter limits the inlet, the eFuse the target rail,"
- moved on the sheet: C104, C105, C106, C107, D102, R101
